File: HW/MainBoard/RevA/FunctionGeneratorCortexM4/AnalogOutput.sch (KiCad schematic (older format))
At the start: 40 parts, among them U11 LTC6910, U12 TL072, U13 TL072, U4 SN74LVC1G3157DCKR, U7 MCP601-xOT

Commit message: Started HW RevB
Parts:
- C26: value CP -> 10uF
Changed lines of the file:
@@
 P 3675 1950
 F 0 "C26" V 3930 1950 50  0000 C CNN
-F 1 "CP" V 3839 1950 50  0000 C CNN
+F 1 "10uF" V 3839 1950 50  0000 C CNN
 F 2 "Capacitor_SMD:CP_Elec_4x5.7" H 3713 1800 50  0001 C CNN
 F 3 "~" H 3675 1950 50  0001 C CNN
