File: HW/MainBoard/RevB/FunctionGeneratorCortexM4/FunctionGeneratorCortexM4.kicad_pcb (KiCad board)
At the start: 2 copper layers, 109.2 x 91.4 mm, 88 parts, among them J1 Conn_02x05_Odd_Even, J2 Screw_Terminal_01x02, J3 Conn_02x06_Odd_Even, J4 Conn_01x06, J5 Conn_01x03, J6 Conn_02x04_Odd_Even, J7 Conn_02x07_Odd_Even, Q1 DMG2301L, U1 NCP51460SN33T1G, U11 LTC6910, U12 TL072, U13 TL072, U2 SN74LVC1G3157DCKR, U3 MCP1703A-3302_SOT223, U4 SN74LVC1G3157DCKR, U5 TC7662Bx0A, U6 STM32G474RET, U7 MCP601-xOT

Commit message: REVB DRAFT LAYOUT
Parts:
- removed TP1: TestPoint, TestPoint:TestPoint_Pad_1.0x1.0mm
- added C27: 10Uf, Capacitor_SMD:C_1206_3216Metric_Pad1.42x1.75mm_HandSolder, F.Cu at (147.4, 67.6)
- added C28: 10Uf, Capacitor_SMD:C_1206_3216Metric_Pad1.42x1.75mm_HandSolder, F.Cu at (162.8, 106.3)
- added C29: 10Uf, Capacitor_SMD:C_1206_3216Metric_Pad1.42x1.75mm_HandSolder, F.Cu at (147.4, 71.2)
- added C30: 1uF, Capacitor_SMD:C_1206_3216Metric_Pad1.42x1.75mm_HandSolder, F.Cu at (131.6, 54.4)
- added C31: 100nF, Capacitor_SMD:C_1206_3216Metric_Pad1.42x1.75mm_HandSolder, F.Cu at (175.8, 63.3)
- added C32: 10uF, Capacitor_SMD:C_1206_3216Metric_Pad1.42x1.75mm_HandSolder, F.Cu at (170.4, 63.3)
- added C33: 100nF, Capacitor_SMD:C_1206_3216Metric_Pad1.42x1.75mm_HandSolder, F.Cu at (160.0, 93.9)
- added C34: 100nF, Capacitor_SMD:C_1206_3216Metric_Pad1.42x1.75mm_HandSolder, F.Cu at (168.1, 93.3)
- added JP3: Jumper_NC_Small, Jumper:SolderJumper-2_P1.3mm_Bridged_Pad1.0x1.5mm, F.Cu at (135.0, 47.8)
- added R22: 1K, Resistor_SMD:R_1206_3216Metric_Pad1.42x1.75mm_HandSolder, F.Cu at (160.3, 57.4)
- added TP12: TestPoint, TestPoint:TestPoint_Pad_1.0x1.0mm, F.Cu at (162.8, 101.6)
- added TP13: TestPoint, TestPoint:TestPoint_Pad_1.0x1.0mm, F.Cu at (168.1, 89.5)
- added TP14: TestPoint, TestPoint:TestPoint_Pad_1.0x1.0mm, F.Cu at (146.1, 109.2)
- added TP15: TestPoint, TestPoint:TestPoint_Pad_1.0x1.0mm, F.Cu at (141.0, 109.2)
- added TP16: TestPoint, TestPoint:TestPoint_Pad_1.0x1.0mm, F.Cu at (154.7, 67.5)
- added U10: TL431DBZ, Package_TO_SOT_SMD:SOT-23, F.Cu at (161.0, 60.7)
- added U8: LM1117-5.0, Package_TO_SOT_SMD:SOT-223-3_TabPin2, F.Cu at (171.9, 56.6)
- added U9: TS12A12511DCNR, Package_TO_SOT_SMD:SOT-23-8_Handsoldering, F.Cu at (162.8, 90.4)
- C1, C11, C12, C2, C3, C5, C6, C7, C8: footprint Capacitor_SMD:C_0805_2012Metric_Pad1.15x1.40mm_HandSolder -> Capacitor_SMD:C_1206_3216Metric_Pad1.42x1.75mm_HandSolder
- C13: value 10uF -> 100nF; footprint Capacitor_SMD:CP_Elec_4x5.7 -> Capacitor_SMD:C_1206_3216Metric_Pad1.42x1.75mm_HandSolder
- C14: value 10uF -> 10Uf; footprint Capacitor_SMD:CP_Elec_4x5.7 -> Capacitor_SMD:C_1206_3216Metric_Pad1.42x1.75mm_HandSolder
- C26: value CP -> 10uF
- J1: footprint Connector_IDC:IDC-Header_2x06_P2.54mm_Vertical -> Connector_IDC:IDC-Header_2x05_P2.54mm_Vertical
- J5: footprint Connector_PinHeader_1.27mm:PinHeader_1x03_P1.27mm_Vertical -> Connector_PinHeader_2.54mm:PinHeader_1x03_P2.54mm_Vertical
- R12: value 100R -> 10K
- R13: value 100R -> 6K2
- R20, R5, R6: value 470R -> 4K7
- U3: value MCP1703A-3302_SOT223 -> LP3992-33B5F; footprint Package_TO_SOT_SMD:SOT-223-3_TabPin2 -> Package_TO_SOT_SMD:TSOT-23-5
- U4: value SN74LVC1G3157DCKR -> NCP1729; footprint Package_TO_SOT_SMD:SOT-363_SC-70-6_Handsoldering -> Package_TO_SOT_SMD:SOT-23-6_Handsoldering
- U5: value TC7662Bx0A -> NCP1729; footprint Package_SO:SOIC-8_3.9x4.9mm_P1.27mm -> Package_TO_SOT_SMD:SOT-23-6_Handsoldering
- moved C14 56.4 mm to (167.8, 110.5)
- moved R5 46.1 mm to (154.8, 51.5), turned to 180 degrees
- moved D2 45.1 mm to (154.8, 48.5), turned to 180 degrees
- moved R6 40.2 mm to (159.3, 106.3)
- moved D3 34.6 mm to (156.5, 106.3), turned to 90 degrees
- moved C25 33.2 mm to (173.0, 104.3), turned to 90 degrees
- moved R13 32.8 mm to (161.6, 67.6)
- moved C26 31.6 mm to (189.4, 73.2), turned to 270 degrees
- moved R12 27.8 mm to (161.6, 65.0), turned to 0 degrees
- moved U4 27.2 mm to (167.8, 105.8), turned to 0 degrees
- moved TP2 25.9 mm to (169.1, 67.2), turned to 180 degrees
- moved R1 24.7 mm to (178.7, 72.9)
- moved R2 24.7 mm to (182.5, 72.9)
- moved TP8 24.7 mm to (175.1, 71.3)
- moved C13 24.5 mm to (147.4, 57.0)
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Connections:
- C13 pad 1: Net-(C13-Pad1) -> /+5V
- C13 pad 2: Net-(C13-Pad2) -> GNDS
- C14 pad 1: GNDS -> Net-(C14-Pad1)
- C14 pad 2: /-5V -> Net-(C14-Pad2)
- D1 pad 1: /+5V -> Net-(C31-Pad1)
- Q1 pad 2: /+5V -> Net-(C31-Pad1)
- R12 pad 1: /AnalogOutput/DCBIAS -> /+2.5V
- R13 pad 1: /AnalogOutput/DCBIAS -> Net-(R12-Pad2)
- R13 pad 2: Net-(R10-Pad1) -> GNDS
- R9 pad 2: Net-(R9-Pad2) -> /MCU/FUNC1_DCBIAS
- TP10 pad 1: /AnalogOutput/DCBIAS -> Net-(TP10-Pad1)
- U11 pad 2: /-5V -> /+2.5V
- U12 pad 1: Net-(R12-Pad2) -> Net-(TP10-Pad1)
- U12 pad 2: Net-(R12-Pad2) -> Net-(TP10-Pad1)
- U12 pad 3: Net-(U12-Pad3) -> /MCU/FUNC1_DCBIAS
- U3 pad 3: /+3V3 -> Net-(JP3-Pad2)
- U4 pad 1: Net-(R9-Pad2) -> /-5V
- U4 pad 2: GNDS -> /+5V
- U4 pad 3: Net-(U12-Pad3) -> Net-(C14-Pad1)
- U4 pad 4: /MCU/FUNC1_DCBIAS -> GNDS
- U4 pad 6: /AnalogOutput/DCBIAS_INVERT_IN -> Net-(C14-Pad2)
- U5 pad 1: /+5V -> /-5V
- U5 pad 2: Net-(C13-Pad1) -> /+5V
- U5 pad 3: GNDS -> Net-(C27-Pad1)
- U5 pad 4: Net-(C13-Pad2) -> GNDS
- U5 pad 5: /-5V -> /+5V
Routing:
- net /+5V: track 276.6 -> 408.7 mm, vias 4 -> 28
- net /+2.5V: track 0.00 -> 34.2 mm
- net Net-(R1-Pad1): track 11.4 -> 42.1 mm
- net Net-(C31-Pad1): track 0.00 -> 27.5 mm
- net /AnalogOutput/DCBIAS_INVERT_IN: track 12.3 -> 38.9 mm, vias 0 -> 2
- net Net-(R10-Pad1): track 8.61 -> 32.3 mm
- net GNDS: track 76.3 -> 95.4 mm, vias 56 -> 42
- net /MCU/FUNC1_DCBIAS: track 13.0 -> 31.9 mm
- net Net-(R9-Pad2): track 16.7 -> 0.00 mm
- net Net-(U12-Pad3): track 16.4 -> 0.00 mm
- net Net-(TP10-Pad1): track 0.00 -> 16.2 mm
- net /-5V: track 103.5 -> 116.0 mm, vias 2 -> 3
- net /AnalogOutput/DCBIAS: track 24.5 -> 12.6 mm
- net /TRIG_SIG_IN: track 51.4 -> 62.0 mm
- net Net-(C13-Pad1): track 10.5 -> 0.00 mm
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- added copper zone on F.Cu, net /+5V
- removed copper zone on F.Cu, net GNDS
Other:
- board text removed: "BYPASS ———>"

Commit message: OPTIMIZED REVB LAYOUT
Parts:
- removed C15, C22: 100nF, Capacitor_SMD:C_1206_3216Metric_Pad1.42x1.75mm_HandSolder
- added C35: 100nF, Capacitor_SMD:C_1206_3216Metric_Pad1.42x1.75mm_HandSolder, F.Cu at (154.4, 87.8)
- added C36: 100nF, Capacitor_SMD:C_1206_3216Metric_Pad1.42x1.75mm_HandSolder, F.Cu at (154.3, 78.9)
- added D5: LED, LED_SMD:LED_1206_3216Metric_Pad1.42x1.75mm_HandSolder, F.Cu at (146.8, 98.8)
- added D6: LED, LED_SMD:LED_1206_3216Metric_Pad1.42x1.75mm_HandSolder, F.Cu at (179.8, 90.3)
- added JP1: Jumper_NC_Small, Jumper:SolderJumper-2_P1.3mm_Bridged_Pad1.0x1.5mm, F.Cu at (158.9, 81.2)
- added JP2: Jumper_NO_Small, Jumper:SolderJumper-2_P1.3mm_Open_Pad1.0x1.5mm, F.Cu at (161.7, 81.2)
- added JP4: Jumper_NO_Small, Jumper:SolderJumper-2_P1.3mm_Open_Pad1.0x1.5mm, F.Cu at (151.1, 115.7)
- added R23: 4K7, Resistor_SMD:R_1206_3216Metric_Pad1.42x1.75mm_HandSolder, F.Cu at (146.8, 94.9)
- added R24: 4K7, Resistor_SMD:R_1206_3216Metric_Pad1.42x1.75mm_HandSolder, F.Cu at (179.8, 85.0)
- added TP1: TestPoint, TestPoint:TestPoint_Pad_1.0x1.0mm, F.Cu at (154.1, 64.1)
- added TP17: TestPoint, TestPoint:TestPoint_Pad_1.0x1.0mm, F.Cu at (179.8, 78.4)
- added U14: NCP1729, Package_TO_SOT_SMD:SOT-23-6_Handsoldering, F.Cu at (175.3, 86.2)
- C13, C25: value 100nF -> 10Uf
- moved C28 44.1 mm to (149.7, 64.1), turned to 0 degrees
- moved C13 44.0 mm to (175.3, 91.1)
- moved C21 41.9 mm to (195.5, 86.9), turned to 90 degrees
- moved U4 40.8 mm to (149.7, 69.2), turned to 270 degrees
- moved C14 40.7 mm to (149.7, 74.0)
- moved R6 38.7 mm to (154.1, 67.9)
- moved U5 34.6 mm to (161.8, 93.8), turned to 0 degrees
- moved D3 33.1 mm to (154.1, 73.3), turned to 270 degrees
- moved C27 32.4 mm to (166.6, 93.7), turned to 90 degrees
- moved C16 28.2 mm to (155.4, 98.8), turned to 180 degrees
- moved TP9 27.4 mm to (201.2, 83.7)
- moved C33 26.4 mm to (184.9, 85.0), turned to 270 degrees
- moved TP11 25.5 mm to (201.2, 89.8)
- moved C29 25.0 mm to (155.4, 94.9), turned to 180 degrees
- moved R2 24.6 mm to (163.2, 88.2), turned to 0 degrees
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Connections:
- C13 pad 1: /+5V -> Net-(C13-Pad1)
- C13 pad 2: GNDS -> Net-(C13-Pad2)
- C16 pad 2: /-5V -> /-5V_DCBIAS
- C25 pad 1: /+5V -> GNDS
- C25 pad 2: GNDS -> /-5V_LPF
- C28 pad 2: /-5V -> /-5V_PGA
- C29 pad 2: /-5V -> /-5V_DCBIAS
- C33 pad 1: /+5V -> /-5V_LPF
- C34 pad 2: /-5V -> /+5V
- R6 pad 1: /-5V -> /-5V_PGA
- TP12 pad 1: /-5V -> /-5V_DCBIAS
- U11 pad 2: /+2.5V -> Net-(JP1-Pad2)
- U11 pad 4: /-5V -> /-5V_PGA
- U12 pad 4: /-5V -> /-5V_DCBIAS
- U13 pad 4: /-5V -> /-5V_LPF
- U4 pad 1: /-5V -> /-5V_PGA
- U5 pad 1: /-5V -> /-5V_DCBIAS
- U9 pad 7: /-5V -> /-5V_DCBIAS
Routing:
- net /+5V: track 408.7 -> 251.2 mm, vias 28 -> 27
- net /-5V: track 116.0 -> 0.00 mm, vias 3 -> 0
- net /-5V_DCBIAS: track 0.00 -> 40.5 mm, vias 0 -> 2
- net Net-(R1-Pad1): track 42.1 -> 6.56 mm
- net /-5V_PGA: track 0.00 -> 26.2 mm
- net Net-(C26-Pad2): track 41.0 -> 66.5 mm, vias 2 -> 0
- net /-5V_LPF: track 0.00 -> 20.8 mm
- net Net-(R10-Pad1): track 32.3 -> 17.9 mm
- net /+2.5V: track 34.2 -> 20.9 mm
- net Net-(C18-Pad2): track 23.4 -> 13.4 mm
- net Net-(JP4-Pad2): track 10.2 -> 19.7 mm
- net /FUNC_SIG_OUT: track 9.65 -> 18.4 mm
- net /MCU/FUNC1_SIG: track 23.0 -> 31.2 mm
- net Net-(JP1-Pad2): track 0.00 -> 7.73 mm
- net Net-(C13-Pad1): track 0.00 -> 7.44 mm
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Other:
- board text added: "CLK"
- board text added: "DCBIAS"
- board text added: "IO"
- board text added: "LPF"
- board text added: "PGA"

Commit message: Final RevB Layout completed
Parts:
- removed J5: Conn_01x03, Connector_PinHeader_2.54mm:PinHeader_1x03_P2.54mm_Vertical
- removed R13: 6K2, Resistor_SMD:R_1206_3216Metric_Pad1.42x1.75mm_HandSolder
- removed TP14, TP15: TestPoint, TestPoint:TestPoint_Pad_1.0x1.0mm
- added C15: 1nF, Capacitor_SMD:C_1206_3216Metric_Pad1.42x1.75mm_HandSolder, F.Cu at (163.1, 60.6)
- added C22: 100nF, Capacitor_SMD:C_1206_3216Metric_Pad1.42x1.75mm_HandSolder, F.Cu at (143.7, 69.1)
- added C37: 100nF, Capacitor_SMD:C_1206_3216Metric_Pad1.42x1.75mm_HandSolder, F.Cu at (161.8, 97.2)
- added C38: 100nF, Capacitor_SMD:C_1206_3216Metric_Pad1.42x1.75mm_HandSolder, F.Cu at (171.6, 86.1)
- added C39: 100nF, Capacitor_SMD:C_1206_3216Metric_Pad1.42x1.75mm_HandSolder, F.Cu at (140.2, 60.1)
- added C40: 100nF, Capacitor_SMD:C_0603_1608Metric_Pad1.05x0.95mm_HandSolder, F.Cu at (121.8, 111.5)
- added C41: 1uF, Capacitor_SMD:C_1206_3216Metric_Pad1.42x1.75mm_HandSolder, F.Cu at (155.9, 73.3)
- added RV1: R_POT_TRIM, Potentiometer_SMD:Potentiometer_Bourns_3314J_Vertical, F.Cu at (163.1, 72.9)
- U14, U4, U5: value NCP1729 -> TPS60400; footprint Package_TO_SOT_SMD:SOT-23-6_Handsoldering -> Package_TO_SOT_SMD:SOT-23-5_HandSoldering
- U2: value SN74LVC1G3157DCKR -> TS5A3357; footprint Package_TO_SOT_SMD:SOT-363_SC-70-6_Handsoldering -> Package_SO:VSSOP-8_2.4x2.1mm_P0.5mm
- moved U2 24.5 mm to (121.5, 108.2), turned to 270 degrees
- moved C12 10.2 mm to (137.1, 89.2)
- moved C1 10.2 mm to (137.1, 81.6)
- moved C11 10.2 mm to (137.1, 86.7)
- moved L1 10.2 mm to (137.1, 84.1)
- moved JP10 8.64 mm to (106.2, 104.8)
- moved R12 6.79 mm to (163.1, 67.6)
- moved U10 6.79 mm to (163.6, 64.1)
- moved R22 6.79 mm to (158.9, 63.8)
- moved L2 5.59 mm to (132.1, 83.3)
- moved C3 5.08 mm to (126.3, 81.9)
- moved C7 5.08 mm to (120.9, 81.9)
- moved C2 5.08 mm to (126.3, 84.5)
- moved C5 5.08 mm to (126.3, 79.4)
- moved C6 5.08 mm to (120.9, 79.4)
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Connections:
- U14 pad 5: /+5V -> Net-(C13-Pad2)
- U2 pad 2: GNDS -> /MCU/COMP1_INP
- U2 pad 3: Net-(J5-Pad2) -> /MCU/ADC_IN3
- U2 pad 4: /TRIG_SIG_IN -> GNDS
- U2 pad 5: /+3V3 -> /MCU/TRIGMUX2
- U2 pad 6: /MCU/CH1_MUX -> /MCU/TRIGMUX1
- U4 pad 5: /+5V -> Net-(C14-Pad2)
- U5 pad 5: /+5V -> Net-(C27-Pad2)
- U6 pad 11: /MCU/CH1_MUX -> Net-(U6-Pad11)
- U6 pad 40: Net-(U6-Pad40) -> /MCU/TRIGMUX1
- U6 pad 41: Net-(U6-Pad41) -> /MCU/TRIGMUX2
Routing:
- net /MCU/CH1_MUX: track 41.3 -> 0.00 mm, vias 2 -> 0
- net /MCU/TRIGMUX1: track 0.00 -> 24.8 mm, vias 0 -> 4
- net /MCU/TRIGMUX2: track 0.00 -> 24.6 mm, vias 0 -> 4
- net /TRIG_SIG_IN: track 58.7 -> 83.2 mm
- net GNDS: track 93.8 -> 113.9 mm, vias 44 -> 50
- net /MCU/TIM2_TF1FP1: track 31.3 -> 13.4 mm, vias 0 -> 2
- net /+5V: track 251.2 -> 268.2 mm
- net /MCU/ADC_IN3: track 31.8 -> 17.2 mm, vias 0 -> 2
- net /+2.5V: track 20.9 -> 33.8 mm
- net /MCU/COMP1_INP: track 27.1 -> 15.3 mm, vias 0 -> 2
- net /PSU/3V3REF: track 9.69 -> 19.8 mm
- net /MCU/BTN1: track 69.1 -> 60.7 mm
- net /MCU/BTN2: track 63.3 -> 55.0 mm
- net /MCU/BTN3: track 57.6 -> 49.6 mm
- net /MCU/BTN4: track 51.6 -> 43.8 mm
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Other:
- board text added: "Adjust to 6K2"
- board text added: "SIGNAL OUT"
- board text added: "STM32G4 Function Generator RevB © C.Sutton"
- board text added: "SYNC OUT"
- board text added: "TRIGGER IN"
- board text removed: "ADC/COMP"
- board text removed: "I/O"
- board text removed: "M4 Function Generator RevA © C.Sutton"
