File: HW/MainBoard/RevB/FunctionGeneratorCortexM4/PSU.sch (KiCad schematic (older format))
At the start: 49 parts, among them Q1 DMG2301L, U1 NCP51460SN33T1G, U10 TL431DBZ, U3 LP3992-33B5F, U4 NCP1729, U5 NCP1729, U6 STM32G474RET, U8 LM1117-5.0

Commit message: REVB DRAFT LAYOUT
Parts:
- removed JP1, JP2: ~SHDN, symbol Device:Jumper_NO_Small
- added R22: 1K, Resistor_SMD:R_1206_3216Metric_Pad1.42x1.75mm_HandSolder, symbol Device:R
- U8: footprint (none) -> Package_TO_SOT_SMD:SOT-223-3_TabPin2
Connections:
- net +2.5V: now also R22.1; no longer C13.1, C25.1, C32.1, C4.1, JP3.1, R5.1, TP2.1, U1.1 (VI), U3.1 (VIN), U4.2 (VIN), U5.2 (VIN), U8.2 (VO)
- net +5V: now reaches U4.5 (~SHDN)
- net +5V: now also C13.1, C25.1, C32.1, C4.1, JP3.1, R5.1, TP2.1, U1.1 (VI), U3.1 (VIN), U4.2 (VIN), U5.2 (VIN), U5.5 (~SHDN), U8.2 (VO), R22.2
Changed lines of the file:
@@
 	1    0    0    -1
 $EndComp
-$Comp
-L Device:Jumper_NO_Small JP2
-U 1 1 5E9D48CF
-P 1425 4025
-F 0 "JP2" H 1425 4100 50  0000 C CNN
-F 1 "~SHDN" H 1425 3925 50  0000 C CNN
-F 2 "" H 1425 4025 50  0001 C CNN
-F 3 "~" H 1425 4025 50  0001 C CNN
-	1    1425 4025
-	1    0    0    -1
-$EndComp
-Wire Wire Line
-	1525 4025 1600 4025
-Wire Wire Line
-	1325 4025 1275 4025
 Connection ~ 1275 4025
 Wire Wire Line
@@
 	1    0    0    -1
 $EndComp
-$Comp
-L Device:Jumper_NO_Small JP1
-U 1 1 5EBFBD08
-P 1150 6175
-F 0 "JP1" H 1150 6250 50  0000 C CNN
-F 1 "~SHDN" H 1150 6075 50  0000 C CNN
-F 2 "" H 1150 6175 50  0001 C CNN
-F 3 "~" H 1150 6175 50  0001 C CNN
-	1    1150 6175
-	1    0    0    -1
-$EndComp
-Wire Wire Line
-	1250 6175 1600 6175
-Wire Wire Line
-	1050 6175 1000 6175
 Connection ~ 1000 6175
 Wire Wire Line
@@
 F 0 "U8" H 2900 1367 50  0000 C CNN
 F 1 "LM1117-5.0" H 2900 1276 50  0000 C CNN
-F 2 "" H 2900 1125 50  0001 C CNN
+F 2 "Package_TO_SOT_SMD:SOT-223-3_TabPin2" H 2900 1125 50  0001 C CNN
 F 3 "http://www.ti.com/lit/ds/symlink/lm1117.pdf" H 2900 1125 50  0001 C CNN
 	1    2900 1125
@@
 F 0 "U10" V 9800 1500 50  0000 C CNN
 F 1 "TL431DBZ" V 9700 1450 50  0000 C CNN
-F 2 "Package_TO_SOT_SMD:SOT-23" H 9900 1550 50  0001 C CIN
+F 2 "Package_TO_SOT_SMD:SOT-23" H 9775 1850 50  0000 C CIN
 F 3 "http://www.ti.com/lit/ds/symlink/tl431.pdf" H 9900 1700 50  0001 C CIN
 	1    9900 1700
@@
 Wire Wire Line
 	9900 1275 9900 1600
-Connection ~ 9250 1275
-Wire Wire Line
-	9250 1275 8675 1275
-Wire Wire Line
-	10450 1275 9900 1275
+Wire Wire Line
+	8650 1275 8200 1275
+Wire Wire Line
+	10450 1275 10275 1275
 $Comp
 L power:GNDS #PWR0111
@@
 Text HLabel 10450 1275 2    50   Input ~ 0
 +2.5V
-Text Label 8675 1275 0    50   ~ 0
+Text Label 8200 1275 0    50   ~ 0
 5V_POL
 Text Notes 2750 825  0    50   ~ 0
 Max Vin: 15V
+$Comp
+L Device:R R?
+U 1 1 5E71CB53
+P 8800 1275
+AR Path="/5EBB9B06/5E71CB53" Ref="R?"  Part="1"
+AR Path="/5E5FDE87/5E71CB53" Ref="R22"  Part="1"
+F 0 "R22" V 8700 1225 50  0000 L CNN
+F 1 "1K" V 8900 1225 50  0000 L CNN
+F 2 "Resistor_SMD:R_1206_3216Metric_Pad1.42x1.75mm_HandSolder" V 8730 1275 50  0001 C CNN
+F 3 "~" H 8800 1275 50  0001 C CNN
+	1    8800 1275
+	0    1    1    0
+$EndComp
+Wire Wire Line
+	8950 1275 9250 1275
+Connection ~ 9250 1275
+$Comp
+L power:PWR_FLAG #FLG0106
+U 1 1 5E73950B
+P 10275 1100
+F 0 "#FLG0106" H 10275 1175 50  0001 C CNN
+F 1 "PWR_FLAG" H 10275 1273 50  0001 C CNN
+F 2 "" H 10275 1100 50  0001 C CNN
+F 3 "~" H 10275 1100 50  0001 C CNN
+	1    10275 1100
+	1    0    0    -1
+$EndComp
+Wire Wire Line
+	10275 1100 10275 1275
+Connection ~ 10275 1275
+Wire Wire Line
+	10275 1275 9900 1275
+Wire Wire Line
+	1000 6175 1600 6175
+Wire Wire Line
+	1275 4025 1600 4025
 $EndSCHEMATC

Commit message: OPTIMIZED REVB LAYOUT
Parts:
- added D5, D6: LED, LED_SMD:LED_1206_3216Metric_Pad1.42x1.75mm_HandSolder, symbol Device:LED
- added R23, R24: 4K7, Resistor_SMD:R_1206_3216Metric_Pad1.42x1.75mm_HandSolder, symbol Device:R
- added TP17: TestPoint, TestPoint:TestPoint_Pad_1.0x1.0mm, symbol Connector:TestPoint
- added U14: NCP1729, Package_TO_SOT_SMD:SOT-23-6_Handsoldering, symbol NCP1729:NCP1729
- C13, C25: value 100nF -> 10Uf
Connections:
- net +5V: now also U14.2 (VIN), U14.5 (~SHDN); no longer C13.1, C25.1
- net GNDS: now also C25.1, D5.2 (A), D6.2 (A), U14.4 (GND); no longer C13.2, C25.2
- net -5V renamed -5V_PGA
- net -5V_PGA: no longer C29.2, TP12.1, U5.1 (VOUT)
- new net: C13.1, U14.3 (C-)
- new net: C13.2, U14.6 (C+)
- new net: D5.1 (K), R23.2
- new net: D6.1 (K), R24.2
- new net -5V_DCBIAS: C29.2, R23.1, TP12.1, U5.1 (VOUT)
- new net -5V_LPF: C25.2, R24.1, TP17.1, U14.1 (VOUT)
Other:
- moved on the sheet: C1, C10, C11, C12, C14, C2, C27, C28, C29, C3, C30, C31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

Commit message: Final RevB Layout completed
Parts:
- removed R13: 6K2, Resistor_SMD:R_1206_3216Metric_Pad1.42x1.75mm_HandSolder, symbol Device:R
- removed U14, U4, U5: NCP1729, Package_TO_SOT_SMD:SOT-23-6_Handsoldering, symbol NCP1729:NCP1729
- added C15: 1nF, Capacitor_SMD:C_1206_3216Metric_Pad1.42x1.75mm_HandSolder, symbol Device:C
- added C22, C37, C38, C39: 100nF, Capacitor_SMD:C_1206_3216Metric_Pad1.42x1.75mm_HandSolder, symbol Device:C
- added RV1: R_POT_TRIM, Potentiometer_SMD:Potentiometer_Bourns_3314J_Vertical, symbol Device:R_POT_TRIM
- added U14, U4, U5: TPS60400, Package_TO_SOT_SMD:SOT-23-5_HandSoldering, symbol TPS6040x:TPS60400
Connections:
- net +2.5V: now also C15.1
- net +5V: now also C22.1, C37.1, C38.1, C39.1, U14.2 (IN), U4.2 (IN), U5.2 (IN)
- net -5V_DCBIAS: now also U5.1 (OUT)
- net -5V_LPF: now also U14.1 (OUT)
- net -5V_PGA: now also U4.1 (OUT)
- net GNDS: now also C15.2, C22.2, C37.2, C38.2, C39.2, RV1.3, U14.4 (GND), U4.4 (GND), U5.4 (GND)
- net at C13.1: now also U14.3 (CFLY-)
- net at C13.2: now also U14.5 (CFLY+)
- net at C14.1: now also U4.3 (CFLY-)
- net at C14.2: now also U4.5 (CFLY+)
- net at C27.1: now also U5.3 (CFLY-)
- net at C27.2: now also U5.5 (CFLY+)
- net at R12.2, U10.2 (REF): now also RV1.1, RV1.2
Other:
- note added: "Adjust to 6K2"
- moved on the sheet: C1, C13, C14, C25, C27, C28, C29, TP17, TP3
