File: HW/ControlsBoard/RevB/ControlsBoard/ControlsBoard.kicad_pcb (KiCad board)
At the start: 2 copper layers, 48.3 x 38.7 mm, 8 parts, among them J1 Conn_02x06_Odd_Even, SW1 Rotary_Encoder_Switch, U1 Tactile_Switch_SPST-NO, U2 Tactile_Switch_SPST-NO, U3 Tactile_Switch_SPST-NO, U4 Tactile_Switch_SPST-NO

Commit message: updated control panel
Parts:
- added REF**: MountingHole_3.2mm_M3, MountingHole:MountingHole_3.2mm_M3, F.Cu at (43.8, 100.8)
- added REF**: MountingHole_3.2mm_M3, MountingHole:MountingHole_3.2mm_M3, F.Cu at (84.8, 100.8)
- added REF**: MountingHole_3.2mm_M3, MountingHole:MountingHole_3.2mm_M3, F.Cu at (43.7, 55.4)
- added REF**: MountingHole_3.2mm_M3, MountingHole:MountingHole_3.2mm_M3, F.Cu at (84.8, 55.4)
- moved J1 0.46 mm to (77.7, 66.5)
Routing:
- net GNDS: track 72.6 -> 93.4 mm, vias 6 -> 4
- net /Controls/BTN2: track 75.2 -> 79.7 mm
- net /Controls/BTN3: track 50.6 -> 52.8 mm
- net /Controls/BTN1: track 98.1 -> 99.8 mm
- net +3V3: track 49.9 -> 50.8 mm
Other:
- board size 48.3 x 38.7 mm -> 48.3 x 52.6 mm
- net class Default: clearance 0.5 -> 0.6
- rule trace_clearance: 0.5 -> 0.6
